File: Prohelion_MotorInterfaceBoardType1/Prohelion_MotorInterfaceBoardType1.kicad_pcb (KiCad board)
At the start: 2 copper layers, 55 x 25 mm, 3 parts

Commit message: mib 3d
Parts:
- removed REF**: Molex_Micro-Fit_3.0_43045-0621_2x03-1MP_P3.00mm_Horizontal, Connector_Molex:Molex_Micro-Fit_3.0_43045-0621_2x03-1MP_P3.00mm_Horizontal
- removed REF**: Molex_Micro-Fit_3.0_43045-0200_2x01_P3.00mm_Horizontal, Connector_Molex:Molex_Micro-Fit_3.0_43045-0200_2x01_P3.00mm_Horizontal
- removed REF**: Molex_Micro-Fit_3.0_43045-1400_2x07_P3.00mm_Horizontal, Connector_Molex:Molex_Micro-Fit_3.0_43045-1400_2x07_P3.00mm_Horizontal
- added J1: Conn_01x14, Connector_Molex:Molex_Micro-Fit_3.0_43045-1400_2x07_P3.00mm_Horizontal, F.Cu at (94.5, 79.5)
- added J2: Conn_01x02, Connector_Molex:Molex_Micro-Fit_3.0_43045-0200_2x01_P3.00mm_Horizontal, F.Cu at (131.2, 62.5)
- added J3: Conn_01x06, Connector_Molex:Molex_Micro-Fit_3.0_43045-0621_2x03-1MP_P3.00mm_Horizontal, F.Cu at (131.0, 72.0)
